File: voltmeter.kicad_pcb (KiCad board)
At the start: 2 copper layers, 96.5 x 26.9 mm, 34 parts, among them CON1 AVR-ISP-6, J1 Conn_01x02, J2 Conn_01x02, J3 Conn_01x01, J4 Conn_01x01, J5 Conn_01x01, J6 Conn_01x01, J7 Conn_01x01, J8 Conn_01x01, J9 Conn_01x01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

Commit message: Commits just before KiCad crashed
Parts:
- turned C5 to 180 degrees
- turned R3 to 180 degrees
- turned R5 to 180 degrees
- turned R6 to 180 degrees
Routing:
- added copper zone on B.Cu, net GND
Other:
- net class Default: clearance 0.2 -> 0.254; trace_width 0.25 -> 0.254; via_dia 0.6 -> 1.6; via_drill 0.4 -> 0.8
- rule trace_clearance: 0.2 -> 0.254
- rule trace_min: 0.2 -> 0.254
- rule via_min_drill: 0.3 -> 0.8
- rule via_min_size: 0.4 -> 1.6
Changed lines of the file:
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@@
   (page A4)
   (layers
-    (0 F.Cu signal)
+    (0 F.Cu signal hide)
     (31 B.Cu signal)
     (32 B.Adhes user hide)
@@
   )
   (setup
-    (last_trace_width 0.25)
-    (trace_clearance 0.2)
+    (last_trace_width 0.254)
+    (trace_clearance 0.254)
     (zone_clearance 0.508)
     (zone_45_only no)
-    (trace_min 0.2)
+    (trace_min 0.254)
     (segment_width 0.2)
     (edge_width 0.15)
-    (via_size 0.6)
-    (via_drill 0.4)
-    (via_min_size 0.4)
-    (via_min_drill 0.3)
+    (via_size 1.6)
+    (via_drill 0.8)
+    (via_min_size 1.6)
+    (via_min_drill 0.8)
     (uvia_size 0.3)
     (uvia_drill 0.1)
@@
   (net 39 "Net-(U2-Pad32)")
   (net_class Default "This is the default net class."
-    (clearance 0.2)
-    (trace_width 0.25)
-    (via_dia 0.6)
-    (via_drill 0.4)
+    (clearance 0.254)
+    (trace_width 0.254)
+    (via_dia 1.6)
+    (via_drill 0.8)
     (uvia_dia 0.3)
     (uvia_drill 0.1)
@@
   )
   (module Capacitors_SMD:C_0805_HandSoldering (layer B.Cu)
-    (at 103.759 97.663)
+    (at 103.759 97.663 180)
     (descr "Capacitor SMD 0805, hand soldering")
     (tags "capacitor 0805")
     (attr smd)
-    (fp_text reference C5 (at 0 1.75) (layer B.SilkS)
-      (effects (font (size 1 1) (thickness 0.15)) (justify mirror))
-    )
-    (fp_text value C (at 0 -1.75) (layer B.Fab)
-      (effects (font (size 1 1) (thickness 0.15)) (justify mirror))
-    )
-    (fp_text user %R (at 0 1.75) (layer B.Fab)
+    (fp_text reference C5 (at 0 1.75 180) (layer B.SilkS)
+      (effects (font (size 1 1) (thickness 0.15)) (justify mirror))
+    )
+    (fp_text value C (at 0 -1.75 180) (layer B.Fab)
+      (effects (font (size 1 1) (thickness 0.15)) (justify mirror))
+    )
+    (fp_text user %R (at 0 1.75 180) (layer B.Fab)
       (effects (font (size 1 1) (thickness 0.15)) (justify mirror))
     )
@@
     (fp_line (start 2.25 -0.87) (end 2.25 0.88) (layer B.CrtYd) (width 0.05))
     (fp_line (start 2.25 -0.87) (end -2.25 -0.87) (layer B.CrtYd) (width 0.05))
-    (pad 1 smd rect (at -1.25 0) (size 1.5 1.25) (layers B.Cu B.Paste B.Mask)
+    (pad 1 smd rect (at -1.25 0 180) (size 1.5 1.25) (layers B.Cu B.Paste B.Mask)
       (net 4 "Net-(C5-Pad1)"))
-    (pad 2 smd rect (at 1.25 0) (size 1.5 1.25) (layers B.Cu B.Paste B.Mask)
+    (pad 2 smd rect (at 1.25 0 180) (size 1.5 1.25) (layers B.Cu B.Paste B.Mask)
       (net 2 GND))
     (model Capacitors_SMD.3dshapes/C_0805.wrl
@@
   )
   (module Resistors_SMD:R_0805_HandSoldering (layer B.Cu)
-    (at 103.759 99.695)
+    (at 103.759 99.695 180)
     (descr "Resistor SMD 0805, hand soldering")
     (tags "resistor 0805")
     (attr smd)
-    (fp_text reference R3 (at 0 1.7) (layer B.SilkS)
-      (effects (font (size 1 1) (thickness 0.15)) (justify mirror))
-    )
-    (fp_text value 1kR (at 0 -1.75) (layer B.Fab)
-      (effects (font (size 1 1) (thickness 0.15)) (justify mirror))
-    )
-    (fp_text user %R (at 0 0) (layer B.Fab)
+    (fp_text reference R3 (at 0 1.7 180) (layer B.SilkS)
+      (effects (font (size 1 1) (thickness 0.15)) (justify mirror))
+    )
+    (fp_text value 1kR (at 0 -1.75 180) (layer B.Fab)
+      (effects (font (size 1 1) (thickness 0.15)) (justify mirror))
+    )
+    (fp_text user %R (at 0 0 180) (layer B.Fab)
       (effects (font (size 0.5 0.5) (thickness 0.075)) (justify mirror))
     )
@@
     (fp_line (start 2.35 -0.9) (end 2.35 0.9) (layer B.CrtYd) (width 0.05))
     (fp_line (start 2.35 -0.9) (end -2.35 -0.9) (layer B.CrtYd) (width 0.05))
-    (pad 1 smd rect (at -1.35 0) (size 1.5 1.3) (layers B.Cu B.Paste B.Mask)
+    (pad 1 smd rect (at -1.35 0 180) (size 1.5 1.3) (layers B.Cu B.Paste B.Mask)
       (net 4 "Net-(C5-Pad1)"))
-    (pad 2 smd rect (at 1.35 0) (size 1.5 1.3) (layers B.Cu B.Paste B.Mask)
+    (pad 2 smd rect (at 1.35 0 180) (size 1.5 1.3) (layers B.Cu B.Paste B.Mask)
       (net 2 GND))
     (model ${KISYS3DMOD}/Resistors_SMD.3dshapes/R_0805.wrl
@@
   )
   (module Resistors_SMD:R_0805_HandSoldering (layer B.Cu)
-    (at 103.759 101.727)
+    (at 103.759 101.727 180)
     (descr "Resistor SMD 0805, hand soldering")
     (tags "resistor 0805")
     (attr smd)
-    (fp_text reference R5 (at 0 1.7) (layer B.SilkS)
-      (effects (font (size 1 1) (thickness 0.15)) (justify mirror))
-    )
-    (fp_text value R (at 0 -1.75) (layer B.Fab)
-      (effects (font (size 1 1) (thickness 0.15)) (justify mirror))
-    )
-    (fp_text user %R (at 0 0) (layer B.Fab)
+    (fp_text reference R5 (at 0 1.7 180) (layer B.SilkS)
+      (effects (font (size 1 1) (thickness 0.15)) (justify mirror))
+    )
+    (fp_text value R (at 0 -1.75 180) (layer B.Fab)
+      (effects (font (size 1 1) (thickness 0.15)) (justify mirror))
+    )
+    (fp_text user %R (at 0 0 180) (layer B.Fab)
       (effects (font (size 0.5 0.5) (thickness 0.075)) (justify mirror))
     )
@@
     (fp_line (start 2.35 -0.9) (end 2.35 0.9) (layer B.CrtYd) (width 0.05))
     (fp_line (start 2.35 -0.9) (end -2.35 -0.9) (layer B.CrtYd) (width 0.05))
-    (pad 1 smd rect (at -1.35 0) (size 1.5 1.3) (layers B.Cu B.Paste B.Mask)
+    (pad 1 smd rect (at -1.35 0 180) (size 1.5 1.3) (layers B.Cu B.Paste B.Mask)
       (net 4 "Net-(C5-Pad1)"))
-    (pad 2 smd rect (at 1.35 0) (size 1.5 1.3) (layers B.Cu B.Paste B.Mask)
+    (pad 2 smd rect (at 1.35 0 180) (size 1.5 1.3) (layers B.Cu B.Paste B.Mask)
       (net 24 "Net-(R5-Pad2)"))
     (model ${KISYS3DMOD}/Resistors_SMD.3dshapes/R_0805.wrl
@@
   )
   (module Resistors_SMD:R_0805_HandSoldering (layer B.Cu)
-    (at 103.839 103.759)
+    (at 103.839 103.759 180)
     (descr "Resistor SMD 0805, hand soldering")
     (tags "resistor 0805")
     (attr smd)
-    (fp_text reference R6 (at 0 1.7) (layer B.SilkS)
-      (effects (font (size 1 1) (thickness 0.15)) (justify mirror))
-    )
-    (fp_text value R (at 0 -1.75) (layer B.Fab)
-      (effects (font (size 1 1) (thickness 0.15)) (justify mirror))
-    )
-    (fp_text user %R (at 0 0) (layer B.Fab)
+    (fp_text reference R6 (at 0 1.7 180) (layer B.SilkS)
+      (effects (font (size 1 1) (thickness 0.15)) (justify mirror))
+    )
+    (fp_text value R (at 0 -1.75 180) (layer B.Fab)
+      (effects (font (size 1 1) (thickness 0.15)) (justify mirror))
+    )
+    (fp_text user %R (at 0 0 180) (layer B.Fab)
       (effects (font (size 0.5 0.5) (thickness 0.075)) (justify mirror))
     )
@@
     (fp_line (start 2.35 -0.9) (end 2.35 0.9) (layer B.CrtYd) (width 0.05))
     (fp_line (start 2.35 -0.9) (end -2.35 -0.9) (layer B.CrtYd) (width 0.05))
-    (pad 1 smd rect (at -1.35 0) (size 1.5 1.3) (layers B.Cu B.Paste B.Mask)
+    (pad 1 smd rect (at -1.35 0 180) (size 1.5 1.3) (layers B.Cu B.Paste B.Mask)
       (net 9 "Net-(J2-Pad1)"))
-    (pad 2 smd rect (at 1.35 0) (size 1.5 1.3) (layers B.Cu B.Paste B.Mask)
+    (pad 2 smd rect (at 1.35 0 180) (size 1.5 1.3) (layers B.Cu B.Paste B.Mask)
       (net 24 "Net-(R5-Pad2)"))
     (model ${KISYS3DMOD}/Resistors_SMD.3dshapes/R_0805.wrl
@@
   (gr_line (start 187.96 93.472) (end 187.96 120.396) (layer Edge.Cuts) (width 0.15))
   (gr_line (start 91.948 93.472) (end 187.96 93.472) (layer Edge.Cuts) (width 0.15))
+  (zone (net 2) (net_name GND) (layer B.Cu) (hatch none 0.508)
+    (connect_pads (clearance 0.254))
+    (min_thickness 0.254)
+    (fill yes (arc_segments 32) (thermal_gap 0.508) (thermal_bridge_width 0.508))
+    (polygon
+      (pts
+        (xy 91.694 93.726) (xy 187.706 93.726) (xy 187.706 120.142) (xy 91.694 120.142)
+      )
+    )
+  )
 )

Commit message: Closing commit
Parts:
- moved J9 4.08 mm to (122.7, 95.8), turned to 45 degrees
- moved R1 3.94 mm to (114.3, 98.8), turned to 90 degrees
- moved J8 3.18 mm to (116.0, 106.0)
- moved J7 3.15 mm to (117.8, 108.5)
- moved J6 3.01 mm to (119.9, 110.7)
- moved C2 1.07 mm to (128.2, 106.6)
- moved Y1 0.30 mm to (129.1, 108.9)
Connections:
- U3 pad 10: Net-(U2-Pad1) -> Net-(U2-Pad30)
- U3 pad 6: Net-(U2-Pad30) -> Net-(U2-Pad1)
- U3 pad 7: Net-(U2-Pad31) -> Net-(U2-Pad32)
- U3 pad 9: Net-(U2-Pad32) -> Net-(U2-Pad31)
- U4 pad 10: Net-(U2-Pad1) -> Net-(U2-Pad30)
- U4 pad 6: Net-(U2-Pad30) -> Net-(U2-Pad1)
- U4 pad 7: Net-(U2-Pad31) -> Net-(U2-Pad32)
- U4 pad 9: Net-(U2-Pad32) -> Net-(U2-Pad31)
- U5 pad 10: Net-(U2-Pad1) -> Net-(U2-Pad30)
- U5 pad 6: Net-(U2-Pad30) -> Net-(U2-Pad1)
- U5 pad 7: Net-(U2-Pad31) -> Net-(U2-Pad32)
- U5 pad 9: Net-(U2-Pad32) -> Net-(U2-Pad31)
- U6 pad 10: Net-(U2-Pad1) -> Net-(U2-Pad30)
- U6 pad 6: Net-(U2-Pad30) -> Net-(U2-Pad1)
- U6 pad 7: Net-(U2-Pad31) -> Net-(U2-Pad32)
- U6 pad 9: Net-(U2-Pad32) -> Net-(U2-Pad31)
Routing:
- net +3V3: track 0.00 -> 42.9 mm
- net Net-(U2-Pad9): track 0.00 -> 24.2 mm
- net Net-(C5-Pad1): track 0.00 -> 23.3 mm
- net /RST: track 0.00 -> 22.3 mm, vias 0 -> 2
- net Net-(U2-Pad10): track 0.00 -> 21.6 mm
- net Net-(U2-Pad11): track 0.00 -> 18.0 mm
- net Net-(U2-Pad2): track 0.00 -> 16.5 mm
- net Net-(U2-Pad1): track 0.00 -> 15.6 mm
- net Net-(CON1-Pad4): track 0.00 -> 13.4 mm, vias 0 -> 2
- net Net-(CON1-Pad3): track 0.00 -> 11.8 mm
- net Net-(U2-Pad32): track 0.00 -> 11.4 mm
- net Net-(J2-Pad1): track 0.00 -> 10.9 mm
- net Net-(C1-Pad1): track 0.00 -> 10.9 mm
- net Net-(CON1-Pad1): track 0.00 -> 10.6 mm
- net Net-(U2-Pad31): track 0.00 -> 6.62 mm
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- added copper zone on B.Cu, net +3V3

Commit message: Update PCB
Parts:
- removed U4, U5, U6: 7SEGMENT_CC, Displays_7-Segment:7SegmentLED_LTS6760_LTS6780
- added D1: 3v6, Diodes_SMD:D_SMA, B.Cu at (30.6, 26.3)
- added R10: 100, Resistors_SMD:R_0805_HandSoldering, B.Cu at (71.8, 38.0)
- added R11: 100, Resistors_SMD:R_0805_HandSoldering, B.Cu at (65.8, 37.3)
- added R12: 100, Resistors_SMD:R_0805_HandSoldering, B.Cu at (63.6, 39.2)
- added R13: 100, Resistors_SMD:R_0805_HandSoldering, B.Cu at (62.4, 43.5)
- added R14: 4K7, Resistors_SMD:R_0805_HandSoldering, B.Cu at (75.0, 31.6)
- added R15: 4K7, Resistors_SMD:R_0805_HandSoldering, B.Cu at (70.2, 31.6)
- added R16: 4K7, Resistors_SMD:R_0805_HandSoldering, B.Cu at (58.8, 28.0)
- added R9: 100, Resistors_SMD:R_0805_HandSoldering, B.Cu at (73.7, 38.0)
- added REF**: 1pin, Connectors:1pin, B.Cu at (21.3, 26.7)
- added REF**: 1pin, Connectors:1pin, B.Cu at (91.6, 45.7)
- C1: value C -> 1U
- C2: value C -> 1u
- C3, C4, C5: value C -> 0.1u
- J9: moved to B.Cu
- Q1, Q2, Q3, Q4: value BC547 -> 2N7002; footprint TO_SOT_Packages_THT:TO-92_Molded_Narrow -> TO_SOT_Packages_SMD:SOT-23; moved to B.Cu
- R1: value R -> 10K
- R2: value R -> 4K7
- R3: value 1kR -> 1K
- R4, R7, R8: value R -> 100
- R5: value R -> 2K2
- R6: value R -> 22K
- U3: value 7SEGMENT_CC -> CA56-12EWA; footprint Displays_7-Segment:7SegmentLED_LTS6760_LTS6780 -> Displays_7-Segment:CA56-12EWA
- Y1: value Crystal -> 16M
- moved U3 133.6 mm to (62.8, 41.3), turned to 90 degrees
- moved R4 129.9 mm to (64.9, 29.5), turned to 270 degrees
- moved Q2 126.8 mm to (73.3, 28.9), turned to 90 degrees
- moved Q1 126.3 mm to (78.9, 41.1), turned to 180 degrees
- moved R2 121.6 mm to (81.7, 40.4), turned to 270 degrees
- moved Q3 118.7 mm to (69.7, 28.9), turned to 90 degrees
- moved R7 117.6 mm to (66.9, 29.5), turned to 270 degrees
- moved Q4 114.3 mm to (61.5, 28.5), turned to 0 degrees
- moved R8 102.9 mm to (78.7, 28.2), turned to 270 degrees
- moved C3 102.3 mm to (40.2, 45.6)
- moved J3 102.0 mm to (33.5, 46.0)
- moved J4 102.0 mm to (29.8, 46.0)
- moved J5 102.0 mm to (37.2, 46.0)
- moved J1 102.0 mm to (23.1, 43.4)
- moved U1 102.0 mm to (34.9, 40.5)
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Connections:
- Q1 pad 2: Net-(Q1-Pad2) -> GND
- Q1 pad 3: GND -> Net-(Q1-Pad3)
- Q2 pad 2: Net-(Q2-Pad2) -> GND
- Q2 pad 3: GND -> Net-(Q2-Pad3)
- Q3 pad 2: Net-(Q3-Pad2) -> GND
- Q3 pad 3: GND -> Net-(Q3-Pad3)
- Q4 pad 2: Net-(Q4-Pad2) -> GND
- Q4 pad 3: GND -> Net-(Q4-Pad3)
- R2 pad 1: Net-(Q1-Pad2) -> Net-(Q1-Pad1)
- R2 pad 2: Net-(R2-Pad2) -> GND
- R4 pad 1: Net-(Q2-Pad2) -> Net-(R4-Pad1)
- R7 pad 1: Net-(Q3-Pad2) -> Net-(R7-Pad1)
- R8 pad 1: Net-(Q4-Pad2) -> Net-(R8-Pad1)
- U2 pad 1: Net-(U2-Pad1) -> Net-(R9-Pad2)
- U2 pad 10: Net-(U2-Pad10) -> Net-(R12-Pad2)
- U2 pad 11: Net-(U2-Pad11) -> Net-(R13-Pad2)
- U2 pad 2: Net-(U2-Pad2) -> Net-(R10-Pad2)
- U2 pad 25: Net-(R2-Pad2) -> Net-(Q1-Pad1)
- U2 pad 26: Net-(R4-Pad2) -> Net-(Q2-Pad1)
- U2 pad 27: Net-(R7-Pad2) -> Net-(Q3-Pad1)
- U2 pad 28: Net-(R8-Pad2) -> Net-(Q4-Pad1)
- U2 pad 30: Net-(U2-Pad30) -> Net-(R4-Pad2)
- U2 pad 31: Net-(U2-Pad31) -> Net-(R7-Pad2)
- U2 pad 32: Net-(U2-Pad32) -> Net-(R8-Pad2)
- U2 pad 9: Net-(U2-Pad9) -> Net-(R11-Pad2)
- U3 pad 1: Net-(U2-Pad11) -> Net-(R13-Pad1)
- U3 pad 10: Net-(U2-Pad30) -> Net-(R7-Pad1)
- U3 pad 2: Net-(U2-Pad10) -> Net-(R12-Pad1)
- U3 pad 3: Net-(Q1-Pad1) -> Net-(R11-Pad1)
- U3 pad 4: Net-(U2-Pad9) -> Net-(R10-Pad1)
- U3 pad 5: Net-(U2-Pad2) -> Net-(R9-Pad1)
- U3 pad 6: Net-(U2-Pad1) -> Net-(Q1-Pad3)
- U3 pad 7: Net-(U2-Pad32) -> Net-(R8-Pad1)
- U3 pad 8: Net-(Q1-Pad1) -> Net-(Q2-Pad3)
- U3 pad 9: Net-(U2-Pad31) -> Net-(Q3-Pad3)
Routing:
- net GND: track 2.28 -> 70.2 mm
- net +3V3: track 42.9 -> 95.7 mm
- net Net-(Q1-Pad1): track 3.94 -> 48.8 mm
- net Net-(R8-Pad2): track 0.00 -> 29.2 mm
- net Net-(Q2-Pad1): track 3.94 -> 31.1 mm
- net Net-(R11-Pad2): track 0.00 -> 26.6 mm
- net Net-(R12-Pad2): track 0.00 -> 25.0 mm
- net Net-(U2-Pad9): track 24.2 -> 0.00 mm
- net Net-(R13-Pad2): track 0.00 -> 23.0 mm
- net Net-(Q3-Pad1): track 3.94 -> 26.7 mm
- net Net-(U2-Pad10): track 21.6 -> 0.00 mm
- net Net-(R9-Pad2): track 0.00 -> 20.4 mm
- net Net-(R10-Pad2): track 0.00 -> 18.9 mm
- net Net-(U2-Pad11): track 18.0 -> 0.00 mm
- net Net-(U2-Pad2): track 16.5 -> 0.00 mm
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Other:
- board size 96.5 x 26.9 mm -> 76.7 x 26.5 mm
- net class Default: clearance 0.254 -> 0.2032
- rule trace_clearance: 0.254 -> 0.2032
