File: voltmeter.sch (KiCad schematic (older format))
At the start: 35 parts, among them CON1 AVR-ISP-6, J1 Conn_01x02, J2 Conn_01x02, J3 Conn_01x01, J4 Conn_01x01, J5 Conn_01x01, J6 Conn_01x01, J7 Conn_01x01, J8 Conn_01x01, J9 Conn_01x01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

Commit message: Closing commit
Connections:
- net at U3.10 (G), U4.10 (G), U5.10 (G)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: now also U2.30 ((PCINT16/RXD)PD0); no longer U2.1 ((PCINT19/OC2B/INT1)PD3)
- net at U3.6 (B), U4.6 (B), U5.6 (B)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: now also U2.1 ((PCINT19/OC2B/INT1)PD3); no longer U2.30 ((PCINT16/RXD)PD0)
- net at U3.7 (A), U4.7 (A), U5.7 (A)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: now also U2.32 ((PCINT18/INT0)PD2); no longer U2.31 ((PCINT17/TXD)PD1)
- net at U3.9 (F), U4.9 (F), U5.9 (F)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: now also U2.31 ((PCINT17/TXD)PD1); no longer U2.32 ((PCINT18/INT0)PD2)
Other:
- note added: "PUT a integrated 4 digit display in this to avoid routing gimmicks\n"
Changed lines of the file:
@@
 LIBS:contrib
 LIBS:valves
+LIBS:voltmeter-cache
 EELAYER 25 0
 EELAYER END
@@
 	6950 3650 4650 3650
 Wire Wire Line
-	6750 3550 6750 4350
-Wire Wire Line
-	6750 3550 4650 3550
-Wire Wire Line
-	6650 3450 6650 4350
-Wire Wire Line
-	6650 3450 4650 3450
-Wire Wire Line
-	6150 3350 6150 4350
-Wire Wire Line
-	6150 3350 4650 3350
-Wire Wire Line
-	4650 3250 6250 3250
-Wire Wire Line
-	6250 3250 6250 4350
+	4650 3350 6650 3350
+Wire Wire Line
+	4650 3250 6750 3250
 Wire Wire Line
 	7150 4350 7150 4250
@@
 	6650 5250 6550 5250
 Connection ~ 6550 5250
+Wire Wire Line
+	6750 3250 6750 4350
+Wire Wire Line
+	6650 3350 6650 4350
+Wire Wire Line
+	6150 3450 6150 4350
+Wire Wire Line
+	6150 3450 4650 3450
+Wire Wire Line
+	6250 3550 6250 4350
+Wire Wire Line
+	6250 3550 4650 3550
+Text Notes 850  5400 0    197  ~ 0
+PUT a integrated 4 digit display in this to avoid routing gimmicks\n
 $EndSCHEMATC

Commit message: Update PCB
Parts:
- removed Q1, Q2, Q3, Q4: BC547, TO_SOT_Packages_THT:TO-92_Molded_Narrow, symbol BC547
- removed U3, U4, U5, U6: 7SEGMENT_CC, Displays_7-Segment:7SegmentLED_LTS6760_LTS6780, symbol 7SEGMENT_CC
- added Q1, Q2, Q3, Q4: 2N7002, TO_SOT_Packages_SMD:SOT-23, symbol 2N7002
- added R10, R11, R12, R13, R9: 100, Resistors_SMD:R_0805_HandSoldering, symbol R
- added R14, R15, R16: 4K7, Resistors_SMD:R_0805_HandSoldering, symbol R
- added U3: CA56-12EWA, Displays_7-Segment:CA56-12EWA, symbol CA56-12EWA
- C1: value C -> 1U
- C2: value C -> 1u
- C3, C4, C5: value C -> 0.1u
- D1: value D_Zener_ALT -> 3v6; footprint (none) -> Diodes_SMD:D_SMA
- R1: value R -> 10K
- R2: value R -> 4K7
- R3: value 1kR -> 1K
- R4, R7, R8: value R -> 100
- R5: value R -> 2K2
- R6: value R -> 22K
- Y1: value Crystal -> 16M
Connections:
- net GND: now also R2.2, Q1.2 (S), Q2.2 (S), Q3.2 (S), Q4.2 (S), R14.2, R15.2, R16.2
- net at U2.1 ((PCINT19/OC2B/INT1)PD3): now also R9.2
- net at U2.10 ((PCINT22/OC0A/AIN0)PD6): now also R12.2
- net at U2.11 ((PCINT23/AIN1)PD7): now also R13.2
- net at U2.2 ((PCINT20/XCK/T0)PD4): now also R10.2
- net at U2.25 ((PCINT10/ADC2)PC2): now also R2.1, Q1.1 (G); no longer R2.2
- net at U2.26 ((PCINT11/ADC3)PC3): now also Q2.1 (G), R14.1; no longer R4.2
- net at U2.27 ((PCINT12/SDA/ADC4)PC4): now also Q3.1 (G), R15.1; no longer R7.2
- net at U2.28 ((PCINT13/SCL/ADC5)PC5): now also Q4.1 (G), R16.1; no longer R8.2
- net at U2.30 ((PCINT16/RXD)PD0): now also R4.2
- net at U2.31 ((PCINT17/TXD)PD1): now also R7.2
- net at U2.32 ((PCINT18/INT0)PD2): now also R8.2
- net at U2.9 ((PCINT21/OC0B/T1)PD5): now also R11.2
- net at R4.1: now also U3.11 (a)
- net at R7.1: now also U3.10 (f)
- net at R8.1: now also U3.7 (b)
- new net: R13.1, U3.1 (e)
- new net: Q4.3 (D), U3.12 (CA1)
- new net: R12.1, U3.2 (d)
- new net: R11.1, U3.3 (DPX)
- new net: R10.1, U3.4 (c)
- new net: R9.1, U3.5 (g)
- new net: Q1.3 (D), U3.6 (CA4)
- new net: Q2.3 (D), U3.8 (CA3)
- new net: Q3.3 (D), U3.9 (CA2)
Other:
- note removed: "PUT a integrated 4 digit display in this to avoid routing gimmicks\n"
- moved on the sheet: C1, C2, C3, C4, C5, CON1, D1, J1, J2, J3, J4, J5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
